File: Project-01-Breadboard-Power-Supply/BreadboardPowerSupply/_restore_backup_2026-07-15T15-19-42-906/BreadboardPowerSupply.kicad_sch (KiCad schematic)
At the start: 17 parts, among them J1 Conn_01x02_Pin, J2 Conn_01x02_Pin, J3 Conn_01x03_Pin, J4 Conn_01x03_Pin, J5 Screw_Terminal_01x02, J6 Barrel_Jack_Switch, J7 Screw_Terminal_01x02, U1 LM7805_TO220, U2 LM317_TO-220

Commit message: Completed first project of Breadboard Power Supply
Connections:
- net PWR_out_top is gone; now on net PWR_output: J1.2 (Pin_2), J3.2 (Pin_2), J5.1 (Pin_1)
- net PWR_out_bottom renamed PWR_output
Changed lines of the file:
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@@
 		)
 	)
-	(label "PWR_out_top"
+	(label "PWR_output"
 		(at 181.61 50.8 0)
 		(effects
@@
 		)
 	)
-	(label "PWR_out_bottom"
+	(label "PWR_output"
 		(at 180.34 91.44 0)
 		(effects
