File: Project-03-MCU-Datalogger-with build-in 512K EEPROM and Clock/MCU-Datalogger-with build-in 512K EEPROM and Clock.kicad_sch (KiCad schematic)
At the start: 0 parts

Commit message: COMPLETED PROJECT
Parts:
- added BT1: Battery, Connector_PinHeader_2.54mm:PinHeader_1x02_P2.54mm_Vertical, symbol Device:Battery
- added C1, C4: 0.1 uf, Capacitor_SMD:C_0805_2012Metric, symbol Device:C
- added C2, C3: 22 pf, Capacitor_SMD:C_0805_2012Metric, symbol Device:C
- added C5: 110 nf, Capacitor_SMD:C_0805_2012Metric, symbol Device:C_Polarized
- added D1, D2: LED, LED_SMD:LED_0805_2012Metric, symbol Device:LED
- added H1, H2, H3, H4: MountingHole, MountingHole:MountingHole_2.1mm, symbol Mechanical:MountingHole
- added R1, R2, R6: 10 kohms, Resistor_SMD:R_0805_2012Metric, symbol Device:R
- added R3, R4: 4.7 kohms, Resistor_SMD:R_0805_2012Metric, symbol Device:R
- added R5, R7: 330 ohms, Resistor_SMD:R_0805_2012Metric, symbol Device:R
- added U1: DS1337S_, DS1337S:SOIC127P600X175-8N, symbol DS1337S_:DS1337S_
- added U2, U3: 24LC1025, Package_SO:SOIC-8_5.3x5.3mm_P1.27mm, symbol Memory_EEPROM:24LC1025
- added U4: ATMEGA328P-AU, ATMEGA:QFP80P900X900X120-32N, symbol ATMEGA328P-AU:ATMEGA328P-AU
- added Y1: 32.768 khz, Crystal:Crystal_SMD_5032-2Pin_5.0x3.2mm_HandSoldering, symbol Device:Crystal
- added Y2: 16 Mhz, Crystal:Crystal_SMD_5032-2Pin_5.0x3.2mm_HandSoldering, symbol Device:Crystal
Connections:
- new net: D1.1 (K), R5.2
- new net: R2.2, U1.7 (SQW/~INT)
- new net: C4.2, U4.20 (AREF)
- new net: D2.1 (K), R7.1
- new net: BT1.1 (+), C5.1, D2.2 (A), U4.18 (AVCC), U4.4 (VCC)
- new net: U1.1 (X1), Y1.2
- new net: U1.2 (X2), Y1.1
- new net: R1.2, U1.3 (~{INTA})
- new net: C3.2, U4.8 (PB7), Y2.1
- new net: C2.2, U4.7 (PB6), Y2.2
- new net D2: U4.32 (PD2)
- new net D3: U4.1 (PD3)
- new net D4: U4.2 (PD4)
- new net D5: U4.9 (PD5)
- new net D6: U4.10 (PD6)
- new net D7: U4.11 (PD7)
- new net D8: U4.12 (PB0)
- new net GND: BT1.2 (-), C1.2, C2.1, C3.1, C4.1, C5.2, R5.1, R7.2, U1.4 (GND), U2.4 (GND), U2.7 (WP), U3.2 (A1), U3.4 (GND), U3.7 (WP), U4.21 (GND), U4.3 (GND), U4.5 (GND)
- new net MISO: U4.16 (PB4)
- new net MOSI: U4.15 (PB3)
- new net RESET: R6.2, U4.29 (PC6/~{RESET})
- new net RX: U4.30 (PD0)
- new net SCK: D1.2 (A), R3.2, U1.6 (SCL), U2.6 (SCL), U3.6 (SCL), U4.17 (PB5), U4.28 (PC5)
- new net SDA: R4.2, U1.5 (SDA), U2.5 (SDA), U3.5 (SDA), U4.27 (PC4)
- new net TX: U4.31 (PD1)
- new net VCC: U4.6 (VCC)
- new net Vcc: C1.1, R1.1, R2.1, R3.1, R4.1, R6.1, U1.8 (VCC), U2.1 (A0), U2.2 (A1), U2.3 (A2), U2.8 (VCC), U3.1 (A0), U3.3 (A2), U3.8 (VCC)
- no-connect marks 0 -> 9
Other:
- added sheet Connectors (connectors.kicad_sch)
- note added: "MCU"
- note added: "MEMORY"
- note added: "MOUNTING HOLES"
- note added: "Real Time Clock"
- title: (none) -> ${project_name}

Commit message: small changes
Connections:
- net Vcc: now also BT1.1 (+), C5.1, D2.2 (A), U4.18 (AVCC), U4.4 (VCC)
Changed lines of the file:
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@@
+		)
+	)
+	(label "Vcc"
+		(at 255.27 34.29 0)
+		(effects
+			(font
+				(size 1.27 1.27)
+			)
+			(justify left bottom)
 		)
 	)

Commit message: small bug correction
Connections:
- net SCK: no longer R3.2, U1.6 (SCL), U2.6 (SCL), U3.6 (SCL), U4.28 (PC5)
- new net SCL: R3.2, U1.6 (SCL), U2.6 (SCL), U3.6 (SCL), U4.28 (PC5)
Other:
- sheet Connectors ports: added SCL; removed none
Changed lines of the file:
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@@
 	(wire
 		(pts
-			(xy 237.49 29.21) (xy 237.49 34.29)
-		)
-		(stroke
-			(width 0)
-			(type default)
-		)
-	)
-	(wire
-		(pts
 			(xy 246.38 54.61) (xy 256.54 54.61)
 		)
@@
 		)
 	)
-	(label "SCK"
+	(label "SCL"
 		(at 100.33 153.67 0)
 		(effects
@@
 		)
 	)
-	(label "SCK"
+	(label "SCL"
 		(at 88.9 147.32 0)
 		(effects
@@
 		)
 	)
-	(label "SCK"
+	(label "SCL"
 		(at 31.75 62.23 0)
 		(effects
@@
 		)
 	)
+	(label "SCK"
+		(at 158.75 151.13 180)
+		(effects
+			(font
+				(size 1.27 1.27)
+			)
+			(justify right bottom)
+		)
+	)
 	(label "Vcc"
 		(at 107.95 134.62 0)
@@
 		)
 	)
-	(label "SCK"
+	(label "SCL"
 		(at 50.8 147.32 0)
 		(effects
@@
 		)
 	)
-	(label "SCK"
+	(label "SCL"
 		(at 195.58 77.47 180)
 		(effects
@@
 		)
 	)
-	(label "SCK"
+	(label "SCL"
 		(at 158.75 128.27 180)
 		(effects
@@
 		)
 	)
-	(symbol
-		(lib_id "power:PWR_FLAG")
-		(at 237.49 29.21 0)
-		(unit 1)
-		(body_style 1)
-		(exclude_from_sim no)
-		(in_bom yes)
-		(on_board yes)
-		(in_pos_files yes)
-		(dnp no)
-		(fields_autoplaced yes)
-		(property "Reference" "#FLG02"
-			(at 237.49 27.305 0)
-			(hide yes)
-			(show_name no)
-			(do_not_autoplace no)
-			(effects
-				(font
-					(size 1.27 1.27)
-				)
-			)
-		)
-		(property "Value" "PWR_FLAG"
-			(at 237.49 24.13 0)
-			(show_name no)
-			(do_not_autoplace no)
-			(effects
-				(font
-					(size 1.27 1.27)
-				)
-			)
-		)
-		(property "Footprint" ""
-			(at 237.49 29.21 0)
-			(hide yes)
-			(show_name no)
-			(do_not_autoplace no)
-			(effects
-				(font
-					(size 1.27 1.27)
-				)
-			)
-		)
-		(property "Datasheet" ""
-			(at 237.49 29.21 0)
-			(hide yes)
-			(show_name no)
-			(do_not_autoplace no)
-			(effects
-				(font
-					(size 1.27 1.27)
-				)
-			)
-		)
-		(property "Description" "Special symbol for telling ERC where power comes from"
-			(at 237.49 29.21 0)
-			(hide yes)
-			(show_name no)
-			(do_not_autoplace no)
-			(effects
-				(font
-					(size 1.27 1.27)
-				)
-			)
-		)
-		(pin "1"
-		)
-		(instances
-			(project "MCU-Datalogger-with build-in 512K EEPROM and Clock"
-				(path "/91329c53-97ad-43cd-a9dd-37636ac44c9f"
-					(reference "#FLG02")
-					(unit 1)
-				)
-			)
-		)
-	)
 	(sheet
 		(at 158.75 109.22)
@@
 			)
 		)
-		(pin "SCK" passive
-			(at 158.75 128.27 180)
+		(pin "SDA" bidirectional
+			(at 158.75 124.46 180)
 			(effects
 				(font
@@
 			)
 		)
-		(pin "SDA" bidirectional
-			(at 158.75 124.46 180)
+		(pin "TX" output
+			(at 158.75 132.08 180)
 			(effects
 				(font
@@
 			)
 		)
-		(pin "TX" output
-			(at 158.75 132.08 180)
+		(pin "Vcc" passive
+			(at 158.75 116.84 180)
 			(effects
 				(font
@@
 			)
 		)
-		(pin "Vcc" passive
-			(at 158.75 116.84 180)
+		(pin "SCK" passive
+			(at 158.75 151.13 180)
+			(effects
+				(font
+					(size 1.27 1.27)
+				)
+				(justify left)
+			)
+		)
+		(pin "SCL" passive
+			(at 158.75 128.27 180)
 			(effects
 				(font
