File: Project-03-MCU-Datalogger-with build-in 512K EEPROM and Clock/connectors.kicad_sch (KiCad schematic)
At the start: 4 parts, among them J1 Conn_01x09_Pin, J2 Conn_01x04_Pin, J4 Conn_02x03_Odd_Even

Commit message: small bug correction
Connections:
- net SCK: no longer J2.4 (Pin_4)
- new net SCL: J2.4 (Pin_4)
Changed lines of the file:
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@@
 		)
 	)
-	(hierarchical_label "SCK"
+	(hierarchical_label "SCL"
 		(shape passive)
 		(at 123.19 88.9 0)
@@
 			)
 		)
-		(property "Description" "UART SERIAL"
+		(property "Description" "I2C"
 			(at 119.38 78.74 0)
 			(show_name no)
@@
 			)
 		)
-		(property "Description" "I2C"
+		(property "Description" "SERIAL"
 			(at 138.43 80.01 0)
 			(show_name no)
